File: esp32-wled-adv-pcb.kicad_pcb (KiCad board)
At the start: 2 copper layers, 39 parts, among them J1 Conn_01x03_Male, J2 Conn_01x03_Male, J3 Barrel_Jack, Q1 BS170F, SW1 SW_Push, SW2 SW_Push, SW3 SW_Push, U1 MT3420C, U2 ESP32-PICO-D4

Commit message: finalize Rev 1
Parts:
- removed J3: Barrel_Jack, Connector_BarrelJack:BarrelJack_Horizontal
- removed SW3: SW_Push, Connector_PinHeader_2.54mm:PinHeader_1x02_P2.54mm_Vertical
- removed TP1: 0.6V, TestPoint:TestPoint_THTPad_D1.0mm_Drill0.5mm
- added C10: 100n, Capacitor_SMD:C_0805_2012Metric, F.Cu at (119.4, 93.3)
- added C11: 100n, Capacitor_SMD:C_0805_2012Metric, F.Cu at (157.9, 111.5)
- added C12: 10µ, Capacitor_SMD:C_0805_2012Metric, F.Cu at (117.1, 97.5)
- added C13: 100n, Capacitor_SMD:C_0805_2012Metric, F.Cu at (114.8, 109.2)
- added C14: 22p, Capacitor_SMD:C_0805_2012Metric, F.Cu at (125.5, 99.4)
- added F1: 5A, Fuse:Fuseholder_Cylinder-5x20mm_Stelvio-Kontek_PTF78_Horizontal_Open, F.Cu at (108.6, 92.2)
- added G***: LOGO, LOGO, F.Cu at (134.0, 89.7)
- added H1: MountingHole, MountingHole:MountingHole_3.2mm_M3_DIN965, F.Cu at (86.2, 126.0)
- added H2: MountingHole, MountingHole:MountingHole_3.2mm_M3_DIN965, F.Cu at (167.8, 126.0)
- added H3: MountingHole, MountingHole:MountingHole_3.2mm_M3_DIN965, F.Cu at (167.8, 91.5)
- added H4: MountingHole, MountingHole:MountingHole_3.2mm_M3_DIN965, F.Cu at (86.2, 91.5)
- added J4: Screw_Terminal_01x02, Footprints:KF103-5.0-2P, F.Cu at (96.9, 110.1)
- added J5: Conn_01x02, Connector_PinHeader_2.54mm:PinHeader_1x02_P2.54mm_Vertical, F.Cu at (162.8, 110.4)
- added R16: 10R, Resistor_SMD:R_0805_2012Metric, F.Cu at (115.7, 112.6)
- C3: value 1µ -> 100n
- C4: value 100n -> 10µ
- C8: value 22µ -> 100n
- C9: value 100n -> 22µ
- J2: footprint Connector_PinHeader_2.54mm:PinHeader_1x03_P2.54mm_Vertical -> Footprints:KF103-5.0-3P
- R15: value 10R -> 4k7
- R3: value 300k -> 4k7
- R4: value 51k -> 300k
- R5: value 15k -> 51k
- R6: value 4k7 -> 15k
- RV1, RV2, RV3: footprint Connector_PinHeader_2.54mm:PinHeader_1x03_P2.54mm_Vertical -> Footprints:Potentiometer_Bourns_PDB181-K415K-x
- moved R8 92.1 mm to (97.0, 120.1), turned to -90 degrees
- moved R9 83.4 mm to (107.0, 120.1), turned to 90 degrees
- moved RV3 78.7 mm to (147.0, 128.0), turned to -90 degrees
- moved RV2 78.6 mm to (122.0, 128.0), turned to -90 degrees
- moved RV1 76.7 mm to (97.0, 128.0), turned to -90 degrees
- moved R12 70.0 mm to (147.0, 120.1), turned to -90 degrees
- moved R10 68.8 mm to (122.0, 120.1), turned to -90 degrees
- moved R11 63.5 mm to (132.0, 120.1), turned to 90 degrees
- moved R4 63.3 mm to (123.3, 99.4), turned to 90 degrees
- moved J2 63.2 mm to (96.9, 95.1), turned to -90 degrees
- moved R13 62.0 mm to (157.0, 120.1), turned to 90 degrees
- moved C7 54.9 mm to (154.3, 104.0), turned to 180 degrees
- moved C9 54.3 mm to (117.1, 93.3), turned to -90 degrees
- moved R1 53.4 mm to (140.1, 95.8), turned to -90 degrees
- moved SW1 52.7 mm to (137.2, 100.8), turned to 90 degrees
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Connections:
- net Net-(AE1-Pad1) renamed /LNA
- C1 pad 1: +5V -> GND
- C1 pad 2: GND -> +5V
- C2 pad 1: GND -> +5V
- C2 pad 2: /RST -> GND
- C3 pad 2: +3V3 -> /RST
- C8 pad 1: +3V3 -> GND
- C8 pad 2: GND -> +3V3
- C9 pad 1: /WLED_CTRL_IO13 -> +3V3
- R10 pad 1: Net-(R10-Pad1) -> +3V3
- R10 pad 2: GND -> Net-(R10-Pad2)
- R11 pad 1: +3V3 -> Net-(R11-Pad1)
- R11 pad 2: Net-(R11-Pad2) -> GND
- R12 pad 1: Net-(R12-Pad1) -> +3V3
- R12 pad 2: GND -> Net-(R12-Pad2)
- R13 pad 1: +3V3 -> Net-(R13-Pad1)
- R13 pad 2: Net-(Q1-Pad2) -> GND
- R14 pad 1: +5V -> +3V3
- R14 pad 2: Net-(Q1-Pad3) -> Net-(Q1-Pad2)
- R15 pad 1: Net-(Q1-Pad3) -> +5V
- R15 pad 2: /LED_DATA -> Net-(Q1-Pad3)
- R2 pad 1: +3V3 -> +5V
- R2 pad 2: /BOOT -> Net-(R2-Pad2)
- R3 pad 2: Net-(R3-Pad2) -> /BOOT
- R4 pad 1: Net-(R3-Pad2) -> +3V3
- R5 pad 2: GND -> Net-(R5-Pad2)
- R6 pad 1: +3V3 -> Net-(R5-Pad2)
- R6 pad 2: /WLED_CTRL_IO13 -> GND
- R7 pad 2: Net-(R7-Pad2) -> /WLED_CTRL_IO13
- R8 pad 1: Net-(R8-Pad1) -> +3V3
- R8 pad 2: GND -> Net-(R8-Pad2)
- R9 pad 1: +3V3 -> Net-(R9-Pad1)
- R9 pad 2: Net-(R9-Pad2) -> GND
- RV1 pad 1: Net-(R7-Pad2) -> Net-(R8-Pad2)
- RV1 pad 2: /WLED_CTRL_IO14 -> /WLED_CTRL_IO25
- RV1 pad 3: Net-(R8-Pad1) -> Net-(R9-Pad1)
- RV2 pad 1: Net-(R9-Pad2) -> Net-(R10-Pad2)
- RV2 pad 2: /WLED_CTRL_IO25 -> /WLED_CTRL_IO26
- RV2 pad 3: Net-(R10-Pad1) -> Net-(R11-Pad1)
- RV3 pad 1: Net-(R11-Pad2) -> Net-(R12-Pad2)
- RV3 pad 2: /WLED_CTRL_IO26 -> /WLED_CTRL_IO14
- RV3 pad 3: Net-(R12-Pad1) -> Net-(R13-Pad1)
- U1 pad 1: +5V -> Net-(R2-Pad2)
- U1 pad 6: Net-(R3-Pad2) -> Net-(R4-Pad2)
Routing:
- net +3V3: track 0.00 -> 195.8 mm, vias 0 -> 15
- net /WLED_CTRL_IO25: track 0.00 -> 67.9 mm
- net /WLED_CTRL_IO26: track 0.00 -> 43.8 mm
- net /WLED_CTRL_IO14: track 0.00 -> 41.3 mm
- net /WLED_CTRL_IO13: track 0.00 -> 39.1 mm
- net Net-(Q1-Pad2): track 0.00 -> 31.4 mm, vias 0 -> 2
- net /LED_DATA: track 0.00 -> 31.1 mm
- net +5V: track 0.00 -> 19.3 mm, vias 0 -> 2
- net /RST: track 0.00 -> 15.3 mm
- net /BOOT: track 0.00 -> 14.8 mm, vias 0 -> 2
- net /ESP_RXD: track 0.00 -> 12.6 mm
- net /ESP_TXD: track 0.00 -> 11.8 mm
- net Net-(Q1-Pad3): track 0.00 -> 10.7 mm
- net Net-(R8-Pad2): track 0.00 -> 7.00 mm
- net Net-(R13-Pad1): track 0.00 -> 7.00 mm
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- added copper zone on B.Cu, net +3V3
- added copper zone on F.Cu, net +3V3
- added copper zone on F.Cu, net +5V
- added copper zone on B.Cu, net /+5Vin
- added copper zone on F.Cu, net /+5Vin
- added copper zone on B.Cu, net GND
- added copper zone on F.Cu, net GND
Other:
- board outline added: 91.5 x 44.5 mm
- board text added: "+5V"
- board text added: "2022 Dirk Riemekasten"
- board text added: "4.0"
- board text added: "DATA"
- board text added: "ESP32 Advanced WLED Board"
- board text added: "E_RXD"
- board text added: "E_TXD"
- board text added: "GND"
- board text added: "JLCJLCJLCJLC"
- board text added: "LED"
- board text added: "POWER"
- board text added: "SW3"
